File: sweeperino.sch (EAGLE design)
At the start: 41 parts, among them IC2 Si570, IC3 LM1117-3.3V, IC5 7805TV, IC6 7805TV, M1 ARDUINO-NANO-3.0, U1 AD8307ARZ, X1 VFO, X2 VFO

Commit message: Updated board
Parts:
- L1: device inductor-neosid:SD12-1000 -> eagle-ltspice:L0204/7
Changed lines of the file:
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@@
 <layer number="97" name="Info" color="7" fill="1" visible="yes" active="yes"/>
 <layer number="98" name="Guide" color="6" fill="1" visible="yes" active="yes"/>
+<layer number="99" name="SpiceOrder" color="5" fill="1" visible="yes" active="yes"/>
 <layer number="101" name="Hidden" color="15" fill="1" visible="yes" active="yes"/>
 <layer number="102" name="Changes" color="12" fill="1" visible="yes" active="yes"/>
@@
 <part name="GND30" library="supply1" deviceset="GND" device=""/>
 <part name="C14" library="rcl" deviceset="C-EU" device="050-024X044" value="0.01"/>
-<part name="L1" library="inductor-neosid" deviceset="SD12" device="-1000"/>
+<part name="L1" library="eagle-ltspice" deviceset="L" device="0204/7"/>
 <part name="R9" library="rcl" deviceset="R-EU_" device="0204/5" value="470"/>
 <part name="C15" library="rcl" deviceset="C-EU" device="050-024X044" value="15"/>
@@
 <instance part="GND30" gate="1" x="-53.34" y="119.38"/>
 <instance part="C14" gate="G$1" x="-147.32" y="91.44" rot="R90"/>
-<instance part="L1" gate="G$1" x="-127" y="91.44"/>
+<instance part="L1" gate="G$1" x="-127" y="91.44" rot="R90"/>
 <instance part="R9" gate="G$1" x="-109.22" y="91.44" rot="R180"/>
 <instance part="C15" gate="G$1" x="-109.22" y="99.06" rot="R90"/>
